File: RealSizes.kicad_sch (KiCad schematic)
At the start: 13 parts

Commit message: added diodes types
Need to ad diff, traces tracks c;learence
Parts:
- removed R1: 0201_0603M, Resistor_SMD:R_0201_0603Metric, symbol Device:R_US
- removed R10: 1812_4532M, Resistor_SMD:R_1812_4532Metric, symbol Device:R_US
- removed R11: 2010_5025M, Resistor_SMD:R_2010_5025Metric, symbol Device:R_US
- removed R12: 2816_7142M, Resistor_SMD:R_2816_7142Metric, symbol Device:R_US
- removed R13: 4020_10251M, Resistor_SMD:R_4020_10251Metric, symbol Device:R_US
- removed R2: 0402_1005M, Resistor_SMD:R_0402_1005Metric, symbol Device:R_US
- removed R3: 0603_1608M, Resistor_SMD:R_0603_1608Metric, symbol Device:R_US
- removed R4: 0805_2012M, Resistor_SMD:R_0805_2012Metric, symbol Device:R_US
- removed R5: 01005_0402M, Resistor_SMD:R_01005_0402Metric, symbol Device:R_US
- removed R6: 1020_2550M, Resistor_SMD:R_1020_2550Metric, symbol Device:R_US
- removed R7: 1206_3216M, Resistor_SMD:R_1206_3216Metric, symbol Device:R_US
- removed R8: 1210_3225M, Resistor_SMD:R_1210_3225Metric, symbol Device:R_US
- removed R9: 1218_3246M, Resistor_SMD:R_1218_3246Metric, symbol Device:R_US

Commit message: added tracks , need to add diff
Parts:
- added R1, R2: R, symbol Device:R
Changed lines of the file:
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@@
 	(generator_version "9.0")
 	(paper "A4")
+	(symbol
+		(lib_id "Device:R")
+		(at 56.515 27.94 90)
+		(unit 1)
+		(exclude_from_sim no)
+		(in_bom yes)
+		(on_board yes)
+		(dnp no)
+		(fields_autoplaced yes)
+		(property "Reference" "R1"
+			(at 56.515 21.59 90)
+			(effects
+				(font
+					(size 1.27 1.27)
+				)
+			)
+		)
+		(property "Value" "R"
+			(at 56.515 24.13 90)
+			(effects
+				(font
+					(size 1.27 1.27)
+				)
+			)
+		)
+		(property "Footprint" ""
+			(at 56.515 29.718 90)
+			(effects
+				(font
+					(size 1.27 1.27)
+				)
+				(hide yes)
+			)
+		)
+		(property "Datasheet" "~"
+			(at 56.515 27.94 0)
+			(effects
+				(font
+					(size 1.27 1.27)
+				)
+				(hide yes)
+			)
+		)
+		(property "Description" "Resistor"
+			(at 56.515 27.94 0)
+			(effects
+				(font
+					(size 1.27 1.27)
+				)
+				(hide yes)
+			)
+		)
+		(pin "1"
+		)
+		(pin "2"
+		)
+		(instances
+			(project ""
+				(path "/87b15cf5-73e3-47ed-8cdf-253a5b2b9752"
+					(reference "R1")
+					(unit 1)
+				)
+			)
+		)
+	)
+	(symbol
+		(lib_id "Device:R")
+		(at 56.515 38.1 90)
+		(unit 1)
+		(exclude_from_sim no)
+		(in_bom yes)
+		(on_board yes)
+		(dnp no)
+		(fields_autoplaced yes)
+		(property "Reference" "R2"
+			(at 56.515 31.75 90)
+			(effects
+				(font
+					(size 1.27 1.27)
+				)
+			)
+		)
+		(property "Value" "R"
+			(at 56.515 34.29 90)
+			(effects
+				(font
+					(size 1.27 1.27)
+				)
+			)
+		)
+		(property "Footprint" ""
+			(at 56.515 39.878 90)
+			(effects
+				(font
+					(size 1.27 1.27)
+				)
+				(hide yes)
+			)
+		)
+		(property "Datasheet" "~"
+			(at 56.515 38.1 0)
+			(effects
+				(font
+					(size 1.27 1.27)
+				)
+				(hide yes)
+			)
+		)
+		(property "Description" "Resistor"
+			(at 56.515 38.1 0)
+			(effects
+				(font
+					(size 1.27 1.27)
+				)
+				(hide yes)
+			)
+		)
+		(pin "2"
+		)
+		(pin "1"
+		)
+		(instances
+			(project ""
+				(path "/87b15cf5-73e3-47ed-8cdf-253a5b2b9752"
+					(reference "R2")
+					(unit 1)
+				)
+			)
+		)
+	)
 	(sheet_instances
 		(path "/"

Commit message: todo
Parts:
- removed R1, R2: R, symbol Device:R
Other:
- note added: "15-10-2025 : SOD-128"
- note added: "To Do List"
Changed lines of the file:
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@@
 	(generator_version "9.0")
 	(paper "A4")
-	(symbol
-		(lib_id "Device:R")
-		(at 56.515 27.94 90)
-		(unit 1)
+	(text "15-10-2025 : \n \n\n\nSOD-128"
 		(exclude_from_sim no)
-		(in_bom yes)
-		(on_board yes)
-		(dnp no)
-		(fields_autoplaced yes)
-		(property "Reference" "R1"
-			(at 56.515 21.59 90)
-			(effects
-				(font
-					(size 1.27 1.27)
-				)
+		(at 45.72 36.195 0)
+		(effects
+			(font
+				(size 1.27 1.27)
+			)
+			(justify left)
+		)
+	)
+	(text "To Do List "
+		(exclude_from_sim no)
+		(at 50.8 28.575 0)
+		(effects
+			(font
+				(size 1.27 1.27)
+				(thickness 0.254)
+				(bold yes)
 			)
 		)
-		(property "Value" "R"
-			(at 56.515 24.13 90)
-			(effects
-				(font
-					(size 1.27 1.27)
-				)
-			)
-		)
-		(property "Footprint" ""
-			(at 56.515 29.718 90)
-			(effects
-				(font
-					(size 1.27 1.27)
-				)
-				(hide yes)
-			)
-		)
-		(property "Datasheet" "~"
-			(at 56.515 27.94 0)
-			(effects
-				(font
-					(size 1.27 1.27)
-				)
-				(hide yes)
-			)
-		)
-		(property "Description" "Resistor"
-			(at 56.515 27.94 0)
-			(effects
-				(font
-					(size 1.27 1.27)
-				)
-				(hide yes)
-			)
-		)
-		(pin "1"
-		)
-		(pin "2"
-		)
-		(instances
-			(project ""
-				(path "/87b15cf5-73e3-47ed-8cdf-253a5b2b9752"
-					(reference "R1")
-					(unit 1)
-				)
-			)
-		)
-	)
-	(symbol
-		(lib_id "Device:R")
-		(at 56.515 38.1 90)
-		(unit 1)
-		(exclude_from_sim no)
-		(in_bom yes)
-		(on_board yes)
-		(dnp no)
-		(fields_autoplaced yes)
-		(property "Reference" "R2"
-			(at 56.515 31.75 90)
-			(effects
-				(font
-					(size 1.27 1.27)
-				)
-			)
-		)
-		(property "Value" "R"
-			(at 56.515 34.29 90)
-			(effects
-				(font
-					(size 1.27 1.27)
-				)
-			)
-		)
-		(property "Footprint" ""
-			(at 56.515 39.878 90)
-			(effects
-				(font
-					(size 1.27 1.27)
-				)
-				(hide yes)
-			)
-		)
-		(property "Datasheet" "~"
-			(at 56.515 38.1 0)
-			(effects
-				(font
-					(size 1.27 1.27)
-				)
-				(hide yes)
-			)
-		)
-		(property "Description" "Resistor"
-			(at 56.515 38.1 0)
-			(effects
-				(font
-					(size 1.27 1.27)
-				)
-				(hide yes)
-			)
-		)
-		(pin "2"
-		)
-		(pin "1"
-		)
-		(instances
-			(project ""
-				(path "/87b15cf5-73e3-47ed-8cdf-253a5b2b9752"
-					(reference "R2")
-					(unit 1)
-				)
-			)
-		)

Commit message: REV1.2
Changes added From Rev1.1
Parts:
- added D2: SMAJ26A, SMAJ26A:DIOM5026X229N, symbol SMAJ26A:SMAJ26A
Changed lines of the file:
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@@
+		)
+	)
+	(symbol
+		(lib_id "SMAJ26A:SMAJ26A")
+		(at 71.755 59.055 0)
+		(unit 1)
+		(exclude_from_sim no)
+		(in_bom yes)
+		(on_board yes)
+		(dnp no)
+		(fields_autoplaced yes)
+		(property "Reference" "D2"
+			(at 71.755 53.34 0)
+			(effects
+				(font
+					(size 1.27 1.27)
+				)
+			)
+		)
+		(property "Value" "SMAJ26A"
+			(at 71.755 55.88 0)
+			(effects
+				(font
+					(size 1.27 1.27)
+				)
+			)
+		)
+		(property "Footprint" "SMAJ26A:DIOM5026X229N"
+			(at 71.755 59.055 0)
+			(effects
+				(font
+					(size 1.27 1.27)
+				)
+				(justify bottom)
+				(hide yes)
+			)
+		)
+		(property "Datasheet" ""
+			(at 71.755 59.055 0)
+			(effects
+				(font
+					(size 1.27 1.27)
+				)
+				(hide yes)
+			)
+		)
+		(property "Description" ""
+			(at 71.755 59.055 0)
+			(effects
+				(font
+					(size 1.27 1.27)
+				)
+				(hide yes)
+			)
+		)
+		(property "DigiKey_Part_Number" "SMAJ26ALFCT-ND"
+			(at 71.755 59.055 0)
+			(effects
+				(font
+					(size 1.27 1.27)
+				)
+				(justify bottom)
+				(hide yes)
+			)
+		)
+		(property "SnapEDA_Link" "https://www.snapeda.com/parts/SMAJ26A/Littelfuse/view-part/?ref=snap"
+			(at 71.755 59.055 0)
+			(effects
+				(font
+					(size 1.27 1.27)
+				)
+				(justify bottom)
+				(hide yes)
+			)
+		)
+		(property "MAXIMUM_PACKAGE_HEIGHT" "2.29 mm"
+			(at 71.755 59.055 0)
+			(effects
+				(font
+					(size 1.27 1.27)
+				)
+				(justify bottom)
+				(hide yes)
+			)
+		)
+		(property "Package" "DO-214 Littelfuse"
+			(at 71.755 59.055 0)
+			(effects
+				(font
+					(size 1.27 1.27)
+				)
+				(justify bottom)
+				(hide yes)
+			)
+		)
+		(property "Check_prices" "https://www.snapeda.com/parts/SMAJ26A/Littelfuse/view-part/?ref=eda"
+			(at 71.755 59.055 0)
+			(effects
+				(font
+					(size 1.27 1.27)
+				)
+				(justify bottom)
+				(hide yes)
+			)
+		)
+		(property "STANDARD" "IPC 7351B"
+			(at 71.755 59.055 0)
+			(effects
+				(font
+					(size 1.27 1.27)
+				)
+				(justify bottom)
+				(hide yes)
+			)
+		)
+		(property "PARTREV" "BA.10/21/20"
+			(at 71.755 59.055 0)
+			(effects
+				(font
+					(size 1.27 1.27)
+				)
+				(justify bottom)
+				(hide yes)
+			)
+		)
+		(property "MF" "Littelfuse"
+			(at 71.755 59.055 0)
+			(effects
+				(font
+					(size 1.27 1.27)
+				)
+				(justify bottom)
+				(hide yes)
+			)
+		)
+		(property "MP" "SMAJ26A"
+			(at 71.755 59.055 0)
+			(effects
+				(font
+					(size 1.27 1.27)
+				)
+				(justify bottom)
+				(hide yes)
+			)
+		)
+		(property "Description_1" "400W Surface Mount Transient Voltage Supressors | Littelfuse SMAJ26A"
+			(at 71.755 59.055 0)
+			(effects
+				(font
+					(size 1.27 1.27)
+				)
+				(justify bottom)
+				(hide yes)
+			)
+		)
+		(property "MANUFACTURER" "Littelfuse"
+			(at 71.755 59.055 0)
+			(effects
+				(font
+					(size 1.27 1.27)
+				)
+				(justify bottom)
+				(hide yes)
+			)
+		)
+		(pin "C"
+		)
+		(pin "A"
+		)
+		(instances
+			(project ""
+				(path "/87b15cf5-73e3-47ed-8cdf-253a5b2b9752"
+					(reference "D2")
+					(unit 1)
+				)
+			)
 		)
 	)
